File: hardware/demo-vigia/demo-vigia.kicad_sch (KiCad schematic)
At the start: 28 parts, among them J1 TYPE-C-31-M-12, J2 SWD, SW1 TS-1187A-B-A-B, U1 STM32G030F6P6, U2 AP2112K-3.3, U3 LM75BD

Commit message: fix: resolve LM75B symbol mismatch in generated schematic
Parts:
- removed U3: LM75BD, Package_SO:SOIC-8_3.9x4.9mm_P1.27mm, symbol Sensor_Temperature:LM75B
- added U3: LM75BD, Package_SO:SOIC-8_3.9x4.9mm_P1.27mm, symbol Sensor_Temperature:LM75C
Connections:
- net +3V3: now also U3.8 (+Vs)
- net GND: now also U3.4 (GND), U3.5 (A2), U3.6 (A1), U3.7 (A0)
- net I2C_SCL: now also U3.2 (SCL)
- net I2C_SDA: now also U3.1 (SDA)
Changed lines of the file:
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@@
 		(instances
 			(project "demo-vigia"
-				(path "/b6957e44-d195-4221-a1b1-24b2de0ac3ba"
+				(path "/88238aff-ddab-4037-a8a5-f1db201c905a"
 					(reference "J1")
 					(unit 1)
@@
 		(instances
 			(project "demo-vigia"
-				(path "/b6957e44-d195-4221-a1b1-24b2de0ac3ba"
+				(path "/88238aff-ddab-4037-a8a5-f1db201c905a"
 					(reference "R5")
 					(unit 1)
@@
 		(instances
 			(project "demo-vigia"
-				(path "/b6957e44-d195-4221-a1b1-24b2de0ac3ba"
+				(path "/88238aff-ddab-4037-a8a5-f1db201c905a"
 					(reference "R6")
 					(unit 1)
@@
 		(instances
 			(project "demo-vigia"
-				(path "/b6957e44-d195-4221-a1b1-24b2de0ac3ba"
+				(path "/88238aff-ddab-4037-a8a5-f1db201c905a"
 					(reference "F1")
 					(unit 1)
@@
 		(instances
 			(project "demo-vigia"
-				(path "/b6957e44-d195-4221-a1b1-24b2de0ac3ba"
+				(path "/88238aff-ddab-4037-a8a5-f1db201c905a"
 					(reference "D2")
 					(unit 1)
@@
 		(instances
 			(project "demo-vigia"
-				(path "/b6957e44-d195-4221-a1b1-24b2de0ac3ba"
+				(path "/88238aff-ddab-4037-a8a5-f1db201c905a"
 					(reference "U2")
 					(unit 1)
@@
 		(instances
 			(project "demo-vigia"
-				(path "/b6957e44-d195-4221-a1b1-24b2de0ac3ba"
+				(path "/88238aff-ddab-4037-a8a5-f1db201c905a"
 					(reference "C1")
 					(unit 1)
@@
 		(instances
 			(project "demo-vigia"
-				(path "/b6957e44-d195-4221-a1b1-24b2de0ac3ba"
+				(path "/88238aff-ddab-4037-a8a5-f1db201c905a"
 					(reference "C2")
 					(unit 1)
@@
 		(instances
 			(project "demo-vigia"
-				(path "/b6957e44-d195-4221-a1b1-24b2de0ac3ba"
+				(path "/88238aff-ddab-4037-a8a5-f1db201c905a"
 					(reference "TP1")
 					(unit 1)
@@
 		(instances
 			(project "demo-vigia"
-				(path "/b6957e44-d195-4221-a1b1-24b2de0ac3ba"
+				(path "/88238aff-ddab-4037-a8a5-f1db201c905a"
 					(reference "TP2")
 					(unit 1)
@@
 		(instances
 			(project "demo-vigia"
-				(path "/b6957e44-d195-4221-a1b1-24b2de0ac3ba"
+				(path "/88238aff-ddab-4037-a8a5-f1db201c905a"
 					(reference "U1")
 					(unit 1)
@@
 		(instances
 			(project "demo-vigia"
-				(path "/b6957e44-d195-4221-a1b1-24b2de0ac3ba"
+				(path "/88238aff-ddab-4037-a8a5-f1db201c905a"
 					(reference "C3")
 					(unit 1)
@@
 		(instances
 			(project "demo-vigia"
-				(path "/b6957e44-d195-4221-a1b1-24b2de0ac3ba"
+				(path "/88238aff-ddab-4037-a8a5-f1db201c905a"
 					(reference "C4")
 					(unit 1)
@@
 		(instances
 			(project "demo-vigia"
-				(path "/b6957e44-d195-4221-a1b1-24b2de0ac3ba"
+				(path "/88238aff-ddab-4037-a8a5-f1db201c905a"
 					(reference "C5")
 					(unit 1)
@@
 		(instances
 			(project "demo-vigia"
-				(path "/b6957e44-d195-4221-a1b1-24b2de0ac3ba"
+				(path "/88238aff-ddab-4037-a8a5-f1db201c905a"
 					(reference "J2")
 					(unit 1)
@@
 	)
 	(symbol
-		(lib_id "Sensor_Temperature:LM75B")
+		(lib_id "Sensor_Temperature:LM75C")
 		(at 45.72 165.1 0)
 		(unit 1)
@@
 		(fields_autoplaced no)
 		(property "Reference" "U3"
-			(at 39.37 176.53 0.0000)
+			(at 39.116 171.45 0.0000)
 			(effects
 				(font
@@
 		)
 		(property "Value" "LM75BD"
-			(at 45.72 176.53 0.0000)
+			(at 47.752 171.45 0.0000)
 			(effects
 				(font
@@
 		)
 		(property "Footprint" "Package_SO:SOIC-8_3.9x4.9mm_P1.27mm"
-			(at 45.72 165.1 0.0000)
+			(at 42.926 165.1 0.0000)
 			(effects
 				(font
@@
 		(instances
 			(project "demo-vigia"
-				(path "/b6957e44-d195-4221-a1b1-24b2de0ac3ba"
+				(path "/88238aff-ddab-4037-a8a5-f1db201c905a"
 					(reference "U3")
 					(unit 1)
@@
 		(instances
 			(project "demo-vigia"
-				(path "/b6957e44-d195-4221-a1b1-24b2de0ac3ba"
+				(path "/88238aff-ddab-4037-a8a5-f1db201c905a"
 					(reference "C6")
 					(unit 1)
@@
 		(instances
 			(project "demo-vigia"
-				(path "/b6957e44-d195-4221-a1b1-24b2de0ac3ba"
+				(path "/88238aff-ddab-4037-a8a5-f1db201c905a"
 					(reference "R1")
 					(unit 1)
@@
 		(instances
 			(project "demo-vigia"
-				(path "/b6957e44-d195-4221-a1b1-24b2de0ac3ba"
+				(path "/88238aff-ddab-4037-a8a5-f1db201c905a"
 					(reference "R2")
 					(unit 1)
@@
 		(instances
 			(project "demo-vigia"
-				(path "/b6957e44-d195-4221-a1b1-24b2de0ac3ba"
+				(path "/88238aff-ddab-4037-a8a5-f1db201c905a"
 					(reference "R3")
 					(unit 1)
@@
 		(instances
 			(project "demo-vigia"
-				(path "/b6957e44-d195-4221-a1b1-24b2de0ac3ba"
+				(path "/88238aff-ddab-4037-a8a5-f1db201c905a"
 					(reference "D1")
 					(unit 1)
@@
 		(instances
 			(project "demo-vigia"
-				(path "/b6957e44-d195-4221-a1b1-24b2de0ac3ba"
+				(path "/88238aff-ddab-4037-a8a5-f1db201c905a"
 					(reference "R4")
 					(unit 1)
@@
 		(instances
 			(project "demo-vigia"
-				(path "/b6957e44-d195-4221-a1b1-24b2de0ac3ba"
+				(path "/88238aff-ddab-4037-a8a5-f1db201c905a"
 					(reference "C7")
 					(unit 1)
@@
 		(instances
 			(project "demo-vigia"
-				(path "/b6957e44-d195-4221-a1b1-24b2de0ac3ba"
+				(path "/88238aff-ddab-4037-a8a5-f1db201c905a"
 					(reference "SW1")
 					(unit 1)
@@
 		(instances
 			(project "demo-vigia"
-				(path "/b6957e44-d195-4221-a1b1-24b2de0ac3ba"
+				(path "/88238aff-ddab-4037-a8a5-f1db201c905a"
 					(reference "#FLG1")
 					(unit 1)
@@
 		(instances
 			(project "demo-vigia"
-				(path "/b6957e44-d195-4221-a1b1-24b2de0ac3ba"
+				(path "/88238aff-ddab-4037-a8a5-f1db201c905a"
 					(reference "#FLG2")
 					(unit 1)
@@
 		(instances
 			(project "demo-vigia"
-				(path "/b6957e44-d195-4221-a1b1-24b2de0ac3ba"
+				(path "/88238aff-ddab-4037-a8a5-f1db201c905a"
 					(reference "#FLG3")
 					(unit 1)
@@
 		(instances
 			(project "demo-vigia"
-				(path "/b6957e44-d195-4221-a1b1-24b2de0ac3ba"
+				(path "/88238aff-ddab-4037-a8a5-f1db201c905a"
 					(reference "H1")
 					(unit 1)
@@
 		(instances
 			(project "demo-vigia"
-				(path "/b6957e44-d195-4221-a1b1-24b2de0ac3ba"
+				(path "/88238aff-ddab-4037-a8a5-f1db201c905a"
 					(reference "H2")
 					(unit 1)
@@
 		(instances
 			(project "demo-vigia"
-				(path "/b6957e44-d195-4221-a1b1-24b2de0ac3ba"
+				(path "/88238aff-ddab-4037-a8a5-f1db201c905a"
 					(reference "H3")
 					(unit 1)
@@
 		(instances
 			(project "demo-vigia"
-				(path "/b6957e44-d195-4221-a1b1-24b2de0ac3ba"
+				(path "/88238aff-ddab-4037-a8a5-f1db201c905a"
 					(reference "H4")
 					(unit 1)
